File: takachi-SPCP0813xx/takachi-SPCP0813xx.kicad_pcb (KiCad board)
At the start: 2 copper layers, 68 x 118 mm, 8 parts

Commit message: 寸法指定を追加
Other:
- board text added: "R10.5mm x 4"
Changed lines of the file:
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@@
+	)
+	(gr_line
+		(start 106.75 38.25)
+		(end 110 42.25)
+		(stroke
+			(width 0.15)
+			(type default)
+		)
+		(layer "User.2")
+	)
+	(gr_line
+		(start 110 41.75)
+		(end 110 42.25)
+		(stroke
+			(width 0.15)
+			(type default)
+		)
+		(layer "User.2")
+	)
+	(gr_line
+		(start 109.5 42.25)
+		(end 110 41.75)
+		(stroke
+			(width 0.15)
+			(type default)
+		)
+		(layer "User.2")
+	)
+	(gr_line
+		(start 110 42.25)
+		(end 109.5 42.25)
+		(stroke
+			(width 0.15)
+			(type default)
+		)
+		(layer "User.2")
 	)
 	(gr_line
@@
 		(layer "User.3")
 	)
+	(gr_text "R10.5mm x 4"
+		(at 101.25 38 0)
+		(layer "User.2")
+		(effects
+			(font
+				(size 1 1)
+				(thickness 0.15)
+			)
+			(justify left bottom)
+		)
+	)
 	(gr_text "Top center corrdinate:\n(X:134 Y:30)"
